Commit message: Add position control in simulation with hard-coded values. Right motor seems to be unstable.

File: ros2_description_bolt/urdf/system_bolt_description.urdf.xacro (robot description, xacro)
@@ -14,5 +14,5 @@
   <xacro:property name="opacity" value="1.0" />
   <xacro:property name="new_leg" value="true" />
-  <xacro:property name="has_passive_ankle" value="true" />
+  <xacro:property name="has_passive_ankle" value="false" />
   <xacro:arg name="prefix" default="" />
   <xacro:arg name="use_crane" default="true" />
@@ -31,5 +31,5 @@
   <gazebo>
     <plugin name="gazebo_ros2_bolt" filename="libgazebo_ros2_control_bolt.so">
-      <parameters>$(find position_velocity_effort_gain_controller)/config/bolt_gazebo_pveg_controller.yaml</parameters>
+      <parameters>$(find gazebo_ros2_control_bolt)/config/bolt_gazebo_config_controller.yaml</parameters>
     </plugin>
   </gazebo>
