Commit message: changement of the ethernet line 4 and 25

File: ros2_description_bolt/ros2_control/system_bolt.ros2_control.xacro (robot description, xacro)
@@ -1,5 +1,5 @@
 <?xml version="1.0"?>
 <robot xmlns:xacro="http://www.ros.org/wiki/xacro">
-  <xacro:macro name="system_bolt_ros2_control" params="name prefix use_sim:=^|false use_fake_hardware:=^|true fake_sensor_commands:=^|false slowdown:=2.0 enp3s0:=^|enp3s0 true:=^|true false:=^|false">
+  <xacro:macro name="system_bolt_ros2_control" params="name prefix use_sim:=^|false use_fake_hardware:=^|true fake_sensor_commands:=^|false slowdown:=2.0 enp6s0f1:=^|enp6s0f1 true:=^|true false:=^|false">
     <ros2_control name="${name}" type="system">
       <xacro:if value="$(arg use_sim)">
@@ -20,5 +20,5 @@
             <param name="example_param_hw_stop_duration_sec">3.0</param>
             <param name="example_param_hw_slowdown">${slowdown}</param>
-            <param name="eth_interface">${enp3s0}</param>
+            <param name="eth_interface">${enp6s0f1}</param>
             <param name="calib_kp">3.</param>
             <param name="calib_kd">0.05</param>
@@ -30,6 +30,6 @@
       <joint name="FLHAA">
         <command_interface name="position">
-          <param name="min">-0.5</param>
-          <param name="max">0.5</param>
+          <param name="min">-0.6</param>
+          <param name="max">0.6</param>
         </command_interface>
         <command_interface name="velocity">

Commit message: changement name variable of ethernet port port to ethernet_port

File: ros2_description_bolt/ros2_control/system_bolt.ros2_control.xacro (robot description, xacro)
@@ -1,5 +1,5 @@
 <?xml version="1.0"?>
 <robot xmlns:xacro="http://www.ros.org/wiki/xacro">
-  <xacro:macro name="system_bolt_ros2_control" params="name prefix use_sim:=^|false use_fake_hardware:=^|true fake_sensor_commands:=^|false slowdown:=2.0 enp6s0f1:=^|enp6s0f1 true:=^|true false:=^|false">
+  <xacro:macro name="system_bolt_ros2_control" params="name prefix use_sim:=^|false use_fake_hardware:=^|true fake_sensor_commands:=^|false slowdown:=2.0 ethernet_port:=^|enp6s0f1 true:=^|true false:=^|false">
     <ros2_control name="${name}" type="system">
       <xacro:if value="$(arg use_sim)">
@@ -20,5 +20,5 @@
             <param name="example_param_hw_stop_duration_sec">3.0</param>
             <param name="example_param_hw_slowdown">${slowdown}</param>
-            <param name="eth_interface">${enp6s0f1}</param>
+            <param name="eth_interface">${ethernet_port}</param>
             <param name="calib_kp">3.</param>
             <param name="calib_kd">0.05</param>
@@ -30,6 +30,6 @@
       <joint name="FLHAA">
         <command_interface name="position">
-          <param name="min">-0.6</param>
-          <param name="max">0.6</param>
+          <param name="min">-0.5</param>
+          <param name="max">0.5</param>
         </command_interface>
         <command_interface name="velocity">

Commit message: fix some last bug from ros2_control_node in the systeme bolt.cpp

File: ros2_description_bolt/ros2_control/system_bolt.ros2_control.xacro (robot description, xacro)
@@ -23,5 +23,5 @@
             <param name="calib_kp">3.</param>
             <param name="calib_kd">0.05</param>
-            <param name="calib_T">2.</param>
+            <param name="calib_T">3.</param>
             <param name="calib_dt">0.001</param>
             </xacro:unless>
@@ -30,4 +30,109 @@
       <joint name="FLHAA">
         <command_interface name="position">
+          <param name="min">-0.9</param>
+          <param name="max">0.9</param>
+        </command_interface>
+        <command_interface name="velocity">
+          <param name="min">-1</param>
+          <param name="max">1</param>
+        </command_interface>
+        <command_interface name="effort">
+          <param name="min">-1</param>
+          <param name="max">1</param>
+        </command_interface>
+        <command_interface name="gain_kp">
+          <param name="min">-1000</param>
+          <param name="max">1000</param>
+        </command_interface>
+        <command_interface name="gain_kd">
+          <param name="min">-1000</param>
+          <param name="max">1000</param>
+        </command_interface>
+        <state_interface name="position"/>
+        <state_interface name="velocity"/>
+        <state_interface name="effort"/>
+        <state_interface name="gain_kp"/>
+        <state_interface name="gain_kd"/>
+        <param name="motor_number">0</param>
+        <param name="gear_ratio">9.</param>
+        <param name="motor_constant">0.025</param>
+        <param name="max_current">12.</param>
+        <param name="max_joint_velocity">80.</param>
+        <param name="safety_damping">0.5</param>
+        <param name="motor_reversed_polarity">${true}</param>
+        <param name="position_offset">0.2393</param>
+      </joint>
+      <joint name="FLHFE">
+        <command_interface name="position">
+          <param name="min">-1.7</param>
+          <param name="max">1.7</param>
+        </command_interface>
+        <command_interface name="velocity">
+          <param name="min">-1</param>
+          <param name="max">1</param>
+        </command_interface>
+        <command_interface name="effort">
+          <param name="min">-1</param>
+          <param name="max">1</param>
+        </command_interface>
+        <command_interface name="gain_kp">
+          <param name="min">-1000</param>
+          <param name="max">1000</param>
+        </command_interface>
+        <command_interface name="gain_kd">
+          <param name="min">-1000</param>
+          <param name="max">1000</param>
+        </command_interface>
+        <state_interface name="position"/>
+        <state_interface name="velocity"/>
+        <state_interface name="effort"/>
+        <state_interface name="gain_kp"/>
+        <state_interface name="gain_kd"/>
+        <param name="motor_number">3</param>
+        <param name="gear_ratio">9.</param>
+        <param name="motor_constant">0.025</param>
+        <param name="max_current">12.</param>
+        <param name="max_joint_velocity">80.</param>
+        <param name="safety_damping">0.5</param>
+        <param name="motor_reversed_polarity">${true}</param>
+        <param name="position_offset">0.3891</param>
+      </joint>
+      <joint name="FLK">
+        <command_interface name="position">
+          <param name="min">-3.4</param>
+          <param name="max">3.4</param>
+        </command_interface>
+        <command_interface name="velocity">
+          <param name="min">-1</param>
+          <param name="max">1</param>
+        </command_interface>
+        <command_interface name="effort">
+          <param name="min">-1</param>
+          <param name="max">1</param>
+        </command_interface>
+        <command_interface name="gain_kp">
+          <param name="min">-1000</param>
+          <param name="max">1000</param>
+        </command_interface>
+        <command_interface name="gain_kd">
+          <param name="min">-1000</param>
+          <param name="max">1000</param>
+        </command_interface>
+        <state_interface name="position"/>
+        <state_interface name="velocity"/>
+        <state_interface name="effort"/>
+        <state_interface name="gain_kp"/>
+        <state_interface name="gain_kd"/>
+        <param name="motor_number">2</param>
+        <param name="gear_ratio">9.</param>
+        <param name="motor_constant">0.025</param>
+        <param name="max_current">12.</param>
+        <param name="max_joint_velocity">80.</param>
+        <param name="safety_damping">0.5</param>
+        <param name="motor_reversed_polarity">${true}</param>
+        <param name="position_offset">0.2745</param>
+      </joint>
+      <joint name="FRHAA">
+        <command_interface name="position">
           <param name="min">-0.5</param>
           <param name="max">0.5</param>
@@ -54,14 +159,14 @@
         <state_interface name="gain_kp"/>
         <state_interface name="gain_kd"/>
-        <param name="motor_number">0</param>
-        <param name="gear_ratio">9.</param>
-        <param name="motor_constant">0.025</param>
-        <param name="max_current">12.</param>
-        <param name="max_joint_velocity">80.</param>
-        <param name="safety_damping">0.5</param>
-        <param name="motor_reversed_polarity">${true}</param>
-        <param name="position_offset">0.238</param>
-      </joint>
-      <joint name="FLHFE">
+        <param name="motor_number">1</param>
+        <param name="gear_ratio">9.</param>
+        <param name="motor_constant">0.025</param>
+        <param name="max_current">12.</param>
+        <param name="max_joint_velocity">80.</param>
+        <param name="safety_damping">0.5</param>
+        <param name="motor_reversed_polarity">${true}</param>
+        <param name="position_offset">0.584</param>
+      </joint>
+      <joint name="FRHFE">
         <command_interface name="position">
           <param name="min">-1.7</param>
@@ -89,14 +194,14 @@
         <state_interface name="gain_kp"/>
         <state_interface name="gain_kd"/>
-        <param name="motor_number">3</param>
-        <param name="gear_ratio">9.</param>
-        <param name="motor_constant">0.025</param>
-        <param name="max_current">12.</param>
-        <param name="max_joint_velocity">80.</param>
-        <param name="safety_damping">0.5</param>
-        <param name="motor_reversed_polarity">${true}</param>
-        <param name="position_offset">-0.308</param>
-      </joint>
-      <joint name="FLK">
+        <param name="motor_number">5</param>
+        <param name="gear_ratio">9.</param>
+        <param name="motor_constant">0.025</param>
+        <param name="max_current">12.</param>
+        <param name="max_joint_velocity">80.</param>
+        <param name="safety_damping">0.5</param>
+        <param name="motor_reversed_polarity">${false}</param>
+        <param name="position_offset">0.09607</param>
+      </joint>
+      <joint name="FRK">
         <command_interface name="position">
           <param name="min">-3.4</param>
@@ -124,75 +229,5 @@
         <state_interface name="gain_kp"/>
         <state_interface name="gain_kd"/>
-        <param name="motor_number">2</param>
-        <param name="gear_ratio">9.</param>
-        <param name="motor_constant">0.025</param>
-        <param name="max_current">12.</param>
-        <param name="max_joint_velocity">80.</param>
-        <param name="safety_damping">0.5</param>
-        <param name="motor_reversed_polarity">${true}</param>
-        <param name="position_offset">0.276</param>
-      </joint>
-      <joint name="FRHAA">
-        <command_interface name="position">
-          <param name="min">-0.5</param>
-          <param name="max">0.5</param>
-        </command_interface>
-        <command_interface name="velocity">
-          <param name="min">-1</param>
-          <param name="max">1</param>
-        </command_interface>
-        <command_interface name="effort">
-          <param name="min">-1</param>
-          <param name="max">1</param>
-        </command_interface>
-        <command_interface name="gain_kp">
-          <param name="min">-1000</param>
-          <param name="max">1000</param>
-        </command_interface>
-        <command_interface name="gain_kd">
-          <param name="min">-1000</param>
-          <param name="max">1000</param>
-        </command_interface>
-        <state_interface name="position"/>
-        <state_interface name="velocity"/>
-        <state_interface name="effort"/>
-        <state_interface name="gain_kp"/>
-        <state_interface name="gain_kd"/>
-        <param name="motor_number">1</param>
-        <param name="gear_ratio">9.</param>
-        <param name="motor_constant">0.025</param>
-        <param name="max_current">12.</param>
-        <param name="max_joint_velocity">80.</param>
-        <param name="safety_damping">0.5</param>
-        <param name="motor_reversed_polarity">${true}</param>
-        <param name="position_offset">-0.115</param>
-      </joint>
-      <joint name="FRHFE">
-        <command_interface name="position">
-          <param name="min">-1.7</param>
-          <param name="max">1.7</param>
-        </command_interface>
-        <command_interface name="velocity">
-          <param name="min">-1</param>
-          <param name="max">1</param>
-        </command_interface>
-        <command_interface name="effort">
-          <param name="min">-1</param>
-          <param name="max">1</param>
-        </command_interface>
-        <command_interface name="gain_kp">
-          <param name="min">-1000</param>
-          <param name="max">1000</param>
-        </command_interface>
-        <command_interface name="gain_kd">
-          <param name="min">-1000</param>
-          <param name="max">1000</param>
-        </command_interface>
-        <state_interface name="position"/>
-        <state_interface name="velocity"/>
-        <state_interface name="effort"/>
-        <state_interface name="gain_kp"/>
-        <state_interface name="gain_kd"/>
-        <param name="motor_number">5</param>
+        <param name="motor_number">4</param>
         <param name="gear_ratio">9.</param>
         <param name="motor_constant">0.025</param>
@@ -201,40 +236,5 @@
         <param name="safety_damping">0.5</param>
         <param name="motor_reversed_polarity">${false}</param>
-        <param name="position_offset">-0.584</param>
-      </joint>
-      <joint name="FRK">
-        <command_interface name="position">
-          <param name="min">-3.4</param>
-          <param name="max">3.4</param>
-        </command_interface>
-        <command_interface name="velocity">
-          <param name="min">-1</param>
-          <param name="max">1</param>
-        </command_interface>
-        <command_interface name="effort">
-          <param name="min">-1</param>
-          <param name="max">1</param>
-        </command_interface>
-        <command_interface name="gain_kp">
-          <param name="min">-1000</param>
-          <param name="max">1000</param>
-        </command_interface>
-        <command_interface name="gain_kd">
-          <param name="min">-1000</param>
-          <param name="max">1000</param>
-        </command_interface>
-        <state_interface name="position"/>
-        <state_interface name="velocity"/>
-        <state_interface name="effort"/>
-        <state_interface name="gain_kp"/>
-        <state_interface name="gain_kd"/>
-        <param name="motor_number">4</param>
-        <param name="gear_ratio">9.</param>
-        <param name="motor_constant">0.025</param>
-        <param name="max_current">12.</param>
-        <param name="max_joint_velocity">80.</param>
-        <param name="safety_damping">0.5</param>
-        <param name="motor_reversed_polarity">${false}</param>
-        <param name="position_offset">0.432</param>
+        <param name="position_offset">0.4386</param>
       </joint>
       <sensor name="IMU">
