Commit message: Change initialisation of bolt. Before we create all the parameters in the xacro, now in the xacro we call config/bolt_config.yaml where we create all paramaters. We also add it in the CMake.

File: ros2_description_bolt/ros2_control/system_bolt.ros2_control.xacro (robot description, xacro)
@@ -17,16 +17,11 @@
           <xacro:unless value="${use_fake_hardware}">
             <plugin>ros2_control_bolt/SystemBoltHardware</plugin>
-            <param name="example_param_hw_start_duration_sec">2.0</param>
-            <param name="example_param_hw_stop_duration_sec">3.0</param>
-            <param name="example_param_hw_slowdown">${slowdown}</param>
-            <param name="eth_interface">${ethernet_port}</param>
-            <param name="calib_kp">3.</param>
-            <param name="calib_kd">0.05</param>
-            <param name="calib_T">3.</param>
-            <param name="calib_dt">0.001</param>
+            <param name="bolt_yaml">2.0</param>
+            <xacro:property name="prop_bolt_config_yaml" value="$(find ros2_description_bolt)/config/bolt_config.yaml" />
+            <param name="bolt_config_yaml">${prop_bolt_config_yaml}</param>
             </xacro:unless>
         </hardware>
       </xacro:unless>
-      <joint name="FLHAA">
+      <!-- <joint name="FLHAA">
         <command_interface name="position">
           <param name="min">-0.9</param>
@@ -61,5 +56,75 @@
         <param name="safety_damping">0.5</param>
         <param name="motor_reversed_polarity">${true}</param>
-        <param name="position_offset">0.2393</param>
+        <param name="position_offset">-0.113570</param>
+      </joint>
+      <joint name="FRHAA">
+        <command_interface name="position">
+          <param name="min">-0.9</param>
+          <param name="max">0.9</param>
+        </command_interface>
+        <command_interface name="velocity">
+          <param name="min">-1</param>
+          <param name="max">1</param>
+        </command_interface>
+        <command_interface name="effort">
+          <param name="min">-1</param>
+          <param name="max">1</param>
+        </command_interface>
+        <command_interface name="gain_kp">
+          <param name="min">-1000</param>
+          <param name="max">1000</param>
+        </command_interface>
+        <command_interface name="gain_kd">
+          <param name="min">-1000</param>
+          <param name="max">1000</param>
+        </command_interface>
+        <state_interface name="position"/>
+        <state_interface name="velocity"/>
+        <state_interface name="effort"/>
+        <state_interface name="gain_kp"/>
+        <state_interface name="gain_kd"/>
+        <param name="motor_number">3</param>
+        <param name="gear_ratio">9.</param>
+        <param name="motor_constant">0.025</param>
+        <param name="max_current">12.</param>
+        <param name="max_joint_velocity">80.</param>
+        <param name="safety_damping">0.5</param>
+        <param name="motor_reversed_polarity">${true}</param>
+        <param name="position_offset">0.834380</param>
+      </joint>
+      <joint name="FLK">
+        <command_interface name="position">
+          <param name="min">-3.4</param>
+          <param name="max">3.4</param>
+        </command_interface>
+        <command_interface name="velocity">
+          <param name="min">-1</param>
+          <param name="max">1</param>
+        </command_interface>
+        <command_interface name="effort">
+          <param name="min">-1</param>
+          <param name="max">1</param>
+        </command_interface>
+        <command_interface name="gain_kp">
+          <param name="min">-1000</param>
+          <param name="max">1000</param>
+        </command_interface>
+        <command_interface name="gain_kd">
+          <param name="min">-1000</param>
+          <param name="max">1000</param>
+        </command_interface>
+        <state_interface name="position"/>
+        <state_interface name="velocity"/>
+        <state_interface name="effort"/>
+        <state_interface name="gain_kp"/>
+        <state_interface name="gain_kd"/>
+        <param name="motor_number">2</param>
+        <param name="gear_ratio">9.</param>
+        <param name="motor_constant">0.025</param>
+        <param name="max_current">12.</param>
+        <param name="max_joint_velocity">80.</param>
+        <param name="safety_damping">0.5</param>
+        <param name="motor_reversed_polarity">${true}</param>
+        <param name="position_offset">-0.058488</param>
       </joint>
       <joint name="FLHFE">
@@ -89,14 +154,14 @@
         <state_interface name="gain_kp"/>
         <state_interface name="gain_kd"/>
-        <param name="motor_number">3</param>
-        <param name="gear_ratio">9.</param>
-        <param name="motor_constant">0.025</param>
-        <param name="max_current">12.</param>
-        <param name="max_joint_velocity">80.</param>
-        <param name="safety_damping">0.5</param>
-        <param name="motor_reversed_polarity">${true}</param>
-        <param name="position_offset">0.3891</param>
-      </joint>
-      <joint name="FLK">
+        <param name="motor_number">1</param>
+        <param name="gear_ratio">9.</param>
+        <param name="motor_constant">0.025</param>
+        <param name="max_current">12.</param>
+        <param name="max_joint_velocity">80.</param>
+        <param name="safety_damping">0.5</param>
+        <param name="motor_reversed_polarity">${true}</param>
+        <param name="position_offset">0.609496</param>
+      </joint>
+      <joint name="FRK">
         <command_interface name="position">
           <param name="min">-3.4</param>
@@ -124,47 +189,12 @@
         <state_interface name="gain_kp"/>
         <state_interface name="gain_kd"/>
-        <param name="motor_number">2</param>
-        <param name="gear_ratio">9.</param>
-        <param name="motor_constant">0.025</param>
-        <param name="max_current">12.</param>
-        <param name="max_joint_velocity">80.</param>
-        <param name="safety_damping">0.5</param>
-        <param name="motor_reversed_polarity">${true}</param>
-        <param name="position_offset">0.2745</param>
-      </joint>
-      <joint name="FRHAA">
-        <command_interface name="position">
-          <param name="min">-0.5</param>
-          <param name="max">0.5</param>
-        </command_interface>
-        <command_interface name="velocity">
-          <param name="min">-1</param>
-          <param name="max">1</param>
-        </command_interface>
-        <command_interface name="effort">
-          <param name="min">-1</param>
-          <param name="max">1</param>
-        </command_interface>
-        <command_interface name="gain_kp">
-          <param name="min">-1000</param>
-          <param name="max">1000</param>
-        </command_interface>
-        <command_interface name="gain_kd">
-          <param name="min">-1000</param>
-          <param name="max">1000</param>
-        </command_interface>
-        <state_interface name="position"/>
-        <state_interface name="velocity"/>
-        <state_interface name="effort"/>
-        <state_interface name="gain_kp"/>
-        <state_interface name="gain_kd"/>
-        <param name="motor_number">1</param>
-        <param name="gear_ratio">9.</param>
-        <param name="motor_constant">0.025</param>
-        <param name="max_current">12.</param>
-        <param name="max_joint_velocity">80.</param>
-        <param name="safety_damping">0.5</param>
-        <param name="motor_reversed_polarity">${true}</param>
-        <param name="position_offset">0.584</param>
+        <param name="motor_number">5</param>
+        <param name="gear_ratio">9.</param>
+        <param name="motor_constant">0.025</param>
+        <param name="max_current">12.</param>
+        <param name="max_joint_velocity">80.</param>
+        <param name="safety_damping">0.5</param>
+        <param name="motor_reversed_polarity">${false}</param>
+        <param name="position_offset">0.093402</param>
       </joint>
       <joint name="FRHFE">
@@ -194,5 +224,5 @@
         <state_interface name="gain_kp"/>
         <state_interface name="gain_kd"/>
-        <param name="motor_number">5</param>
+        <param name="motor_number">4</param>
         <param name="gear_ratio">9.</param>
         <param name="motor_constant">0.025</param>
@@ -201,41 +231,6 @@
         <param name="safety_damping">0.5</param>
         <param name="motor_reversed_polarity">${false}</param>
-        <param name="position_offset">0.09607</param>
-      </joint>
-      <joint name="FRK">
-        <command_interface name="position">
-          <param name="min">-3.4</param>
-          <param name="max">3.4</param>
-        </command_interface>
-        <command_interface name="velocity">
-          <param name="min">-1</param>
-          <param name="max">1</param>
-        </command_interface>
-        <command_interface name="effort">
-          <param name="min">-1</param>
-          <param name="max">1</param>
-        </command_interface>
-        <command_interface name="gain_kp">
-          <param name="min">-1000</param>
-          <param name="max">1000</param>
-        </command_interface>
-        <command_interface name="gain_kd">
-          <param name="min">-1000</param>
-          <param name="max">1000</param>
-        </command_interface>
-        <state_interface name="position"/>
-        <state_interface name="velocity"/>
-        <state_interface name="effort"/>
-        <state_interface name="gain_kp"/>
-        <state_interface name="gain_kd"/>
-        <param name="motor_number">4</param>
-        <param name="gear_ratio">9.</param>
-        <param name="motor_constant">0.025</param>
-        <param name="max_current">12.</param>
-        <param name="max_joint_velocity">80.</param>
-        <param name="safety_damping">0.5</param>
-        <param name="motor_reversed_polarity">${false}</param>
-        <param name="position_offset">0.4386</param>
-      </joint>
+        <param name="position_offset">0.586886</param>
+      </joint> -->
       <sensor name="IMU">
         <state_interface name="gyroscope_x"/>
@@ -255,6 +250,6 @@
         <state_interface name="attitude_quaternion_z"/>
         <state_interface name="attitude_quaternion_w"/>
-        <param name="rotate_vector">1 2 3</param>
-        <param name="orientation_vector">1 2 3 4</param>
+        <!-- <param name="rotate_vector">1 2 3</param>
+        <param name="orientation_vector">1 2 3 4</param> -->
       </sensor>
     </ros2_control>

Commit message: restore definition of each joints and delete the informations whe doesn't need because they are already in the yaml file

File: ros2_description_bolt/ros2_control/system_bolt.ros2_control.xacro (robot description, xacro)
@@ -23,5 +23,5 @@
         </hardware>
       </xacro:unless>
-      <!-- <joint name="FLHAA">
+      <joint name="FLHAA">
         <command_interface name="position">
           <param name="min">-0.9</param>
@@ -49,12 +49,4 @@
         <state_interface name="gain_kp"/>
         <state_interface name="gain_kd"/>
-        <param name="motor_number">0</param>
-        <param name="gear_ratio">9.</param>
-        <param name="motor_constant">0.025</param>
-        <param name="max_current">12.</param>
-        <param name="max_joint_velocity">80.</param>
-        <param name="safety_damping">0.5</param>
-        <param name="motor_reversed_polarity">${true}</param>
-        <param name="position_offset">-0.113570</param>
       </joint>
       <joint name="FRHAA">
@@ -84,12 +76,4 @@
         <state_interface name="gain_kp"/>
         <state_interface name="gain_kd"/>
-        <param name="motor_number">3</param>
-        <param name="gear_ratio">9.</param>
-        <param name="motor_constant">0.025</param>
-        <param name="max_current">12.</param>
-        <param name="max_joint_velocity">80.</param>
-        <param name="safety_damping">0.5</param>
-        <param name="motor_reversed_polarity">${true}</param>
-        <param name="position_offset">0.834380</param>
       </joint>
       <joint name="FLK">
@@ -119,12 +103,4 @@
         <state_interface name="gain_kp"/>
         <state_interface name="gain_kd"/>
-        <param name="motor_number">2</param>
-        <param name="gear_ratio">9.</param>
-        <param name="motor_constant">0.025</param>
-        <param name="max_current">12.</param>
-        <param name="max_joint_velocity">80.</param>
-        <param name="safety_damping">0.5</param>
-        <param name="motor_reversed_polarity">${true}</param>
-        <param name="position_offset">-0.058488</param>
       </joint>
       <joint name="FLHFE">
@@ -154,12 +130,4 @@
         <state_interface name="gain_kp"/>
         <state_interface name="gain_kd"/>
-        <param name="motor_number">1</param>
-        <param name="gear_ratio">9.</param>
-        <param name="motor_constant">0.025</param>
-        <param name="max_current">12.</param>
-        <param name="max_joint_velocity">80.</param>
-        <param name="safety_damping">0.5</param>
-        <param name="motor_reversed_polarity">${true}</param>
-        <param name="position_offset">0.609496</param>
       </joint>
       <joint name="FRK">
@@ -189,12 +157,4 @@
         <state_interface name="gain_kp"/>
         <state_interface name="gain_kd"/>
-        <param name="motor_number">5</param>
-        <param name="gear_ratio">9.</param>
-        <param name="motor_constant">0.025</param>
-        <param name="max_current">12.</param>
-        <param name="max_joint_velocity">80.</param>
-        <param name="safety_damping">0.5</param>
-        <param name="motor_reversed_polarity">${false}</param>
-        <param name="position_offset">0.093402</param>
       </joint>
       <joint name="FRHFE">
@@ -224,13 +184,5 @@
         <state_interface name="gain_kp"/>
         <state_interface name="gain_kd"/>
-        <param name="motor_number">4</param>
-        <param name="gear_ratio">9.</param>
-        <param name="motor_constant">0.025</param>
-        <param name="max_current">12.</param>
-        <param name="max_joint_velocity">80.</param>
-        <param name="safety_damping">0.5</param>
-        <param name="motor_reversed_polarity">${false}</param>
-        <param name="position_offset">0.586886</param>
-      </joint> -->
+      </joint>
       <sensor name="IMU">
         <state_interface name="gyroscope_x"/>

Commit message: change the path of the files names, for match to our link

File: ros2_description_bolt/ros2_control/system_bolt.ros2_control.xacro (robot description, xacro)
@@ -23,5 +23,5 @@
         </hardware>
       </xacro:unless>
-      <joint name="FLHAA">
+      <joint name="FL_HAA">
         <command_interface name="position">
           <param name="min">-0.9</param>
@@ -50,5 +50,5 @@
         <state_interface name="gain_kd"/>
       </joint>
-      <joint name="FRHAA">
+      <joint name="FR_HAA">
         <command_interface name="position">
           <param name="min">-0.9</param>
@@ -77,5 +77,5 @@
         <state_interface name="gain_kd"/>
       </joint>
-      <joint name="FLK">
+      <joint name="FL_KFE">
         <command_interface name="position">
           <param name="min">-3.4</param>
@@ -104,5 +104,5 @@
         <state_interface name="gain_kd"/>
       </joint>
-      <joint name="FLHFE">
+      <joint name="FR_KFE">
         <command_interface name="position">
           <param name="min">-1.7</param>
@@ -131,5 +131,5 @@
         <state_interface name="gain_kd"/>
       </joint>
-      <joint name="FRK">
+      <joint name="FL_HFE">
         <command_interface name="position">
           <param name="min">-3.4</param>
@@ -158,5 +158,5 @@
         <state_interface name="gain_kd"/>
       </joint>
-      <joint name="FRHFE">
+      <joint name="FR_HFE">
         <command_interface name="position">
           <param name="min">-1.7</param>

Commit message: Modifications on doc + Modification of order of joints on yaml files and ros2_description_bolt + adding system_interface_odri.hpp (1) - Maybe new changes

File: ros2_description_bolt/ros2_control/system_bolt.ros2_control.xacro (robot description, xacro)
@@ -23,6 +23,6 @@
             <param name="odri_config_yaml">${prop_bolt_config_yaml}</param>
             <param name="desired_starting_position">0.0 0.0 0.0 0.0 0.0 0.0</param>
-            <param name="default_joint_cmd">FL_HAA 0.0 0.0 0.0 3.0 0.05 FR_HAA 0.0 0.0 0.0 3.0 0.05 FL_KFE 0.0 0.0 0.0 3.0 0.05 FL_HFE 0.0 0.0 0.0 3.0 0.05 FR_KFE 0.0 0.0 0.0 3.0 0.05 FR_HFE 0.0 0.0 0.0 3.0 0.05</param>
-            <param name="default_joint_state">FL_HAA 0.0 0.0 0.0 3.0 0.05 FR_HAA 0.0 0.0 0.0 3.0 0.05 FL_KFE 0.0 0.0 0.0 3.0 0.05 FL_HFE 0.0 0.0 0.0 3.0 0.05 FR_KFE 0.0 0.0 0.0 3.0 0.05 FR_HFE 0.0 0.0 0.0 3.0 0.05</param>
+            <param name="default_joint_cmd">FL_HAA 0.0 0.0 0.0 3.0 0.05 FR_HAA 0.0 0.0 0.0 3.0 0.05 FL_HFE 0.0 0.0 0.0 3.0 0.05 FR_HFE 0.0 0.0 0.0 3.0 0.05 FL_KFE 0.0 0.0 0.0 3.0 0.05 FR_KFE 0.0 0.0 0.0 3.0 0.05</param>
+            <param name="default_joint_state">FL_HAA 0.0 0.0 0.0 3.0 0.05 FR_HAA 0.0 0.0 0.0 3.0 0.05 FL_HFE 0.0 0.0 0.0 3.0 0.05 FR_HFE 0.0 0.0 0.0 3.0 0.05 FL_KFE 0.0 0.0 0.0 3.0 0.05 FR_KFE 0.0 0.0 0.0 3.0 0.05</param>
          </xacro:unless>
         </hardware>
@@ -82,5 +82,5 @@
         <state_interface name="gain_kd"/>
       </joint>
-      <joint name="FL_KFE">
+      <joint name="FL_HFE">
         <command_interface name="position">
           <param name="min">-3.4</param>
@@ -109,5 +109,5 @@
         <state_interface name="gain_kd"/>
       </joint>
-      <joint name="FR_KFE">
+      <joint name="FR_HFE">
         <command_interface name="position">
           <param name="min">-1.7</param>
@@ -136,5 +136,5 @@
         <state_interface name="gain_kd"/>
       </joint>
-      <joint name="FL_HFE">
+      <joint name="FL_KFE">
         <command_interface name="position">
           <param name="min">-3.4</param>
@@ -163,5 +163,5 @@
         <state_interface name="gain_kd"/>
       </joint>
-      <joint name="FR_HFE">
+      <joint name="FR_KFE">
         <command_interface name="position">
           <param name="min">-1.7</param>
